File: PCB_source/AS5601_BreakoutBoard_V1_0.sch (KiCad schematic (older format))
At the start: 8 parts, among them P1 CONN_01X07, P2 MountHole_M3, P3 MountHole_M3, U1 AS5601

Commit message: add step and refactoring
Parts:
- C1, C2: footprint Capacitors_SMD:C_0603_HandSoldering -> footprints:C_0603_HandSoldering; symbol C_Small -> Device:C_Small
- P1: footprint user:USER_SIL-7 -> footprints:USER_SIL-7; symbol CONN_01X07 -> AS5601_breakout:CONN_01X07
- P2, P3: symbol CONN_01X01 -> AS5601_breakout:CONN_01X01
- R1, R2: footprint Resistors_SMD:R_0603_HandSoldering -> footprints:R_0603_HandSoldering; symbol R_Small -> Device:R_Small
- U1: footprint Housings_SOIC:SOIC-8_3.9x4.9mm_Pitch1.27mm -> footprints:SOIC-8_3.9x4.9mm_Pitch1.27mm; symbol AS5601 -> AS5601_breakout:AS5601
Connections:
- wire segments 33 -> 34
Changed lines of the file:
@@
-EESchema Schematic File Version 2
-LIBS:74xgxx
-LIBS:74xx
-LIBS:ac-dc
-LIBS:actel
-LIBS:adc-dac
-LIBS:Altera
-LIBS:analog_devices
-LIBS:analog_switches
-LIBS:atmel
-LIBS:audio
-LIBS:brooktre
-LIBS:cmos_ieee
-LIBS:cmos4000
-LIBS:conn
-LIBS:contrib
-LIBS:cypress
-LIBS:dc-dc
-LIBS:device
-LIBS:digital-audio
-LIBS:diode
-LIBS:display
-LIBS:dsp
-LIBS:elec-unifil
-LIBS:ESD_Protection
-LIBS:ftdi
-LIBS:gennum
-LIBS:graphic
-LIBS:hc11
-LIBS:intel
-LIBS:interface
-LIBS:ir
-LIBS:Lattice
-LIBS:linear
-LIBS:logo
-LIBS:maxim
-LIBS:memory
-LIBS:microchip
-LIBS:microchip_dspic33dsc
-LIBS:microchip_pic10mcu
-LIBS:microchip_pic12mcu
-LIBS:microchip_pic16mcu
-LIBS:microchip_pic18mcu
-LIBS:microchip_pic32mcu
-LIBS:microcontrollers
-LIBS:motor_drivers
-LIBS:motorola
-LIBS:msp430
-LIBS:nordicsemi
-LIBS:nxp_armmcu
-LIBS:onsemi
-LIBS:opto
-LIBS:Oscillators
-LIBS:philips
-LIBS:power
-LIBS:Power_Management
-LIBS:powerint
-LIBS:pspice
-LIBS:references
-LIBS:regul
-LIBS:relays
-LIBS:rfcom
-LIBS:sensors
-LIBS:silabs
-LIBS:siliconi
-LIBS:stm8
-LIBS:stm32
-LIBS:supertex
-LIBS:switches
-LIBS:texas
-LIBS:transf
-LIBS:transistors
-LIBS:ttl_ieee
-LIBS:user
-LIBS:valves
-LIBS:video
-LIBS:Xicor
-LIBS:xilinx
-LIBS:Zilog
-LIBS:Logo_DirRot_v01
-LIBS:AS5601_v02-cache
-EELAYER 25 0
+EESchema Schematic File Version 4
+EELAYER 30 0
 EELAYER END
 $Descr A4 11693 8268
@@
 $EndDescr
 $Comp
-L AS5601 U1
+L AS5601_breakout:AS5601 U1
 U 1 1 594F3E3A
 P 2450 1800
 F 0 "U1" H 2450 1550 60  0000 C CNN
 F 1 "AS5601" H 2450 2050 50  0000 C CNN
-F 2 "Housings_SOIC:SOIC-8_3.9x4.9mm_Pitch1.27mm" H 2450 2050 60  0001 C CNN
+F 2 "footprints:SOIC-8_3.9x4.9mm_Pitch1.27mm" H 2450 2050 60  0001 C CNN
 F 3 "" H 2450 2050 60  0000 C CNN
 	1    2450 1800
@@
 $EndComp
 $Comp
-L CONN_01X07 P1
+L AS5601_breakout:CONN_01X07 P1
 U 1 1 594F3E81
 P 800 1650
 F 0 "P1" H 800 2050 50  0000 C CNN
 F 1 "CONN_01X07" V 900 1650 50  0000 C CNN
-F 2 "user:USER_SIL-7" H 800 1650 50  0001 C CNN
-F 3 "http://akizukidenshi.com/catalog/g/gC-09862/" H 800 1650 50  0001 C CNN
+F 2 "footprints:USER_SIL-7" H 800 1650 50  0001 C CNN
+F 3 "" H 800 1650 50  0001 C CNN
 	1    800  1650
 	-1   0    0    -1
 $EndComp
 $Comp
-L +5V #PWR01
+L power:+5V #PWR01
 U 1 1 594F3F87
 P 1100 1300
@@
 $EndComp
 $Comp
-L +3.3V #PWR02
+L power:+3.3V #PWR02
 U 1 1 594F3FA3
 P 1300 1300
@@
 	1300 1450 1300 1300
 $Comp
-L GND #PWR03
+L power:GND #PWR03
 U 1 1 594F3FC5
 P 1300 1950
@@
 	1300 1550 1300 1950
 $Comp
-L +5V #PWR04
+L power:+5V #PWR04
 U 1 1 594F402D
 P 2000 1600
@@
 	2000 1650 2050 1650
 $Comp
-L +3.3V #PWR05
+L power:+3.3V #PWR05
 U 1 1 594F4048
 P 1800 1600
@@
 	1800 1750 2050 1750
 $Comp
-L GND #PWR06
+L power:GND #PWR06
 U 1 1 594F4065
 P 2000 2000
@@
 A
 $Comp
-L R_Small R1
+L Device:R_Small R1
 U 1 1 594F42E7
 P 3200 1600
 F 0 "R1" H 3230 1620 50  0000 L CNN
 F 1 "3.9k" H 3230 1560 50  0000 L CNN
-F 2 "Resistors_SMD:R_0603_HandSoldering" H 3200 1600 50  0001 C CNN
+F 2 "footprints:R_0603_HandSoldering" H 3200 1600 50  0001 C CNN
 F 3 "" H 3200 1600 50  0001 C CNN
 	1    3200 1600
@@
 $EndComp
 $Comp
-L C_Small C1
+L Device:C_Small C1
 U 1 1 594F4454
 P 2350 1050
 F 0 "C1" H 2360 1120 50  0000 L CNN
 F 1 "0.1u" H 2360 970 50  0000 L CNN
-F 2 "Capacitors_SMD:C_0603_HandSoldering" H 2350 1050 50  0001 C CNN
-F 3 "http://akizukidenshi.com/catalog/g/gP-05616/" H 2350 1050 50  0001 C CNN
+F 2 "footprints:C_0603_HandSoldering" H 2350 1050 50  0001 C CNN
+F 3 "" H 2350 1050 50  0001 C CNN
 	1    2350 1050
 	1    0    0    -1
 $EndComp
 $Comp
-L C_Small C2
+L Device:C_Small C2
 U 1 1 594F4545
 P 2600 1050
 F 0 "C2" H 2610 1120 50  0000 L CNN
 F 1 "1u" H 2610 970 50  0000 L CNN
-F 2 "Capacitors_SMD:C_0603_HandSoldering" H 2600 1050 50  0001 C CNN
-F 3 "http://akizukidenshi.com/catalog/g/gP-09348/" H 2600 1050 50  0001 C CNN
+F 2 "footprints:C_0603_HandSoldering" H 2600 1050 50  0001 C CNN
+F 3 "" H 2600 1050 50  0001 C CNN
 	1    2600 1050
 	1    0    0    -1
 $EndComp
 $Comp
-L +5V #PWR07
+L power:+5V #PWR07
 U 1 1 594F4835
 P 2350 900
@@
 $EndComp
 $Comp
-L GND #PWR08
+L power:GND #PWR08
 U 1 1 594F48CE
 P 2350 1200
@@
 	2350 950  2350 900
 $Comp
-L +3.3V #PWR09
+L power:+3.3V #PWR09
 U 1 1 594F49EC
 P 2600 900
@@
 	2600 1150 2600 1200
 $Comp
-L GND #PWR010
+L power:GND #PWR010
 U 1 1 594F4A5F
 P 2600 1200
@@
 	3200 1750 3200 1700
 $Comp
-L R_Small R2
+L Device:R_Small R2
 U 1 1 594F4FF9
 P 3450 1600
 F 0 "R2" H 3480 1620 50  0000 L CNN
 F 1 "3.9k" H 3480 1560 50  0000 L CNN
-F 2 "Resistors_SMD:R_0603_HandSoldering" H 3450 1600 50  0001 C CNN
+F 2 "footprints:R_0603_HandSoldering" H 3450 1600 50  0001 C CNN
 F 3 "" H 3450 1600 50  0001 C CNN
 	1    3450 1600
@@
 	3450 1850 3450 1700
 Wire Wire Line
-	3200 1450 3450 1450
+	3200 1450 3300 1450
 Wire Wire Line
 	3450 1450 3450 1500
@@
 Connection ~ 3300 1450
 $Comp
-L +5V #PWR011
+L power:+5V #PWR011
 U 1 1 594F5320
 P 3300 1300
@@
 	3300 1300 3300 1450
 $Comp
-L PWR_FLAG #FLG012
+L power:PWR_FLAG #FLG012
 U 1 1 594F5CE6
 P 800 2950
@@
 $EndComp
 $Comp
-L +5V #PWR013
+L power:+5V #PWR013
 U 1 1 594F5E14
 P 800 2900
@@
 $EndComp
 $Comp
-L +3.3V #PWR014
+L power:+3.3V #PWR014
 U 1 1 594F5EEF
 P 1150 2900
@@
 $EndComp
 $Comp
-L GND #PWR015
+L power:GND #PWR015
 U 1 1 594F5FB2
 P 1500 3000
@@
 $EndComp
 $Comp
-L PWR_FLAG #FLG016
+L power:PWR_FLAG #FLG016
 U 1 1 594F6015
 P 1150 2950
@@
 $EndComp
 $Comp
-L PWR_FLAG #FLG017
+L power:PWR_FLAG #FLG017
 U 1 1 594F605A
 P 1500 2900
@@
 	800  2950 800  2900
 $Comp
-L CONN_01X01 P2
+L AS5601_breakout:CONN_01X01 P2
 U 1 1 59741010
 P 900 3600
@@
 $EndComp
 $Comp
-L CONN_01X01 P3
+L AS5601_breakout:CONN_01X01 P3
 U 1 1 59741205
 P 900 3800
@@
 Text Label 2950 1950 0    60   ~ 0
 B
+Wire Wire Line
+	3300 1450 3450 1450
 $EndSCHEMATC
